File: Documentation/Cosmic_Game.kicad_sch (KiCad schematic)
At the start: 5 parts, among them J1 ADXL345, J2 Rotary_Encoder, J3 OLED_Screen, J4 NeoPixel_LED, U1 Xiao ESP32C3

Commit message: Add files via upload
Parts:
- added BAT1: LiPo Battery, symbol Connector_Generic:Conn_01x02
- added SW1: Power_Switch, symbol Switch:SW_SPST
Connections:
- net GND: now also BAT1.2 (Pin_2)
- net +5V_IN: now reaches U1.12 (Pin_12)
- net +5V_IN: now also SW1.2 (B)
- new net: BAT1.1 (Pin_1), SW1.1 (A)
